Commit message: fix: reconstruir xacro desde archivos frescos del target con solo 3 cambios: package name, _joint removal, joint rename

File: Laboratorio No. 05 - Robótica de Desarrollo ROS Jazzy y Phantom Pincher X100/pincher_description/urdf/phantomx_pincher_arm.xacro (robot description, xacro)
@@ -66,4 +66,5 @@
     <xacro:gripper_finger_base prefix="${prefix}" parent="gripper_servo_link" name="gripper_finger_base" joint_origin_xyz="0 ${ax12_width/2} 0.0" joint_origin_rpy="${pi} 0.0 ${pi/2}" collision="${collision}" gazebo_preserve_fixed_joint="${gazebo_preserve_fixed_joint}"/>
     <xacro:pincher_finger prefix="${prefix}" parent="gripper_finger_base_link" name="gripper_finger1" joint_origin_xyz="${finger_centre_offset_x} ${finger_centre_offset_y} 0.0" joint_origin_rpy="${pi/2} 0.0 ${pi/2}" collision="${collision}" gazebo_preserve_fixed_joint="${gazebo_preserve_fixed_joint}" mimic_joint="${prefix}gripper" mimic_multiplier="0.005" mimic_offset="0.001"/>
+    <!-- If enabled, mimic finger joints -->
     <xacro:if value="${mimic_finger_joints}">
       <xacro:pincher_finger prefix="${prefix}" parent="gripper_finger_base_link" name="gripper_finger2" joint_origin_xyz="${finger_centre_offset_x} ${-finger_centre_offset_y} 0.0" joint_origin_rpy="${pi/2} ${pi} ${pi/2}" collision="${collision}" gazebo_preserve_fixed_joint="${gazebo_preserve_fixed_joint}" mimic_joint="${prefix}gripper_finger1"/>

File: Laboratorio No. 05 - Robótica de Desarrollo ROS Jazzy y Phantom Pincher X100/pincher_description/urdf/phantomx_pincher_hardware.xacro (robot description, xacro)
@@ -189,17 +189,17 @@
   <xacro:property name="pincher_finger_link_mesh" value="finger"/>
   <xacro:property name="pincher_finger_link_collision_type" value="mesh"/>
-   <xacro:macro name="pincher_finger" params="
-     prefix
-     name
-     parent
-     joint_origin_xyz
-     joint_origin_rpy
-     collision:=true
-     mimic_joint:=none
-     mimic_multiplier:=1.0
-     mimic_offset:=0.0
-     gazebo_preserve_fixed_joint:=false
-   ">
-     <xacro:phantomx_pincher_joint parent="${prefix}${parent}" child="${prefix}${name}_link" joint_name="${prefix}${name}" joint_type="${pincher_finger_joint_type}" joint_origin_xyz="${joint_origin_xyz}" joint_origin_rpy="${joint_origin_rpy}" joint_axis_xyz="${pincher_finger_joint_axis_xyz}" joint_lower_limit="${pincher_finger_joint_lower_limit}" joint_upper_limit="${pincher_finger_joint_upper_limit}" joint_velocity_limit="${pincher_finger_joint_velocity_limit}" joint_torque_limit="${pincher_finger_joint_torque_limit}" joint_damping="${pincher_finger_joint_damping}" joint_friction="${pincher_finger_joint_friction}" gazebo_preserve_fixed_joint="${gazebo_preserve_fixed_joint}" mimic_joint="${mimic_joint}" mimic_multiplier="${mimic_multiplier}" mimic_offset="${mimic_offset}"/>
+  <xacro:macro name="pincher_finger" params="
+    prefix
+    name
+    parent
+    joint_origin_xyz
+    joint_origin_rpy
+    collision:=true
+    mimic_joint:=none
+    mimic_multiplier:=1.0
+    mimic_offset:=0.0
+    gazebo_preserve_fixed_joint:=false
+  ">
+    <xacro:phantomx_pincher_joint parent="${prefix}${parent}" child="${prefix}${name}_link" joint_name="${prefix}${name}" joint_type="${pincher_finger_joint_type}" joint_origin_xyz="${joint_origin_xyz}" joint_origin_rpy="${joint_origin_rpy}" joint_axis_xyz="${pincher_finger_joint_axis_xyz}" joint_lower_limit="${pincher_finger_joint_lower_limit}" joint_upper_limit="${pincher_finger_joint_upper_limit}" joint_velocity_limit="${pincher_finger_joint_velocity_limit}" joint_torque_limit="${pincher_finger_joint_torque_limit}" joint_damping="${pincher_finger_joint_damping}" joint_friction="${pincher_finger_joint_friction}" gazebo_preserve_fixed_joint="${gazebo_preserve_fixed_joint}" mimic_joint="${mimic_joint}" mimic_multiplier="${mimic_multiplier}" mimic_offset="${mimic_offset}"/>
     <xacro:phantomx_pincher_link link_name="${prefix}${name}_link" mesh="${pincher_finger_link_mesh}" collision="${collision}" collision_type="${pincher_finger_link_collision_type}" mu="${pincher_finger_link_mu}"/>
   </xacro:macro>

File: Laboratorio No. 05 - Robótica de Desarrollo ROS Jazzy y Phantom Pincher X100/pincher_description/urdf/phantomx_pincher_utils.xacro (robot description, xacro)
@@ -58,22 +58,22 @@
   <!-- Macro -->
   <!--       -->
-   <xacro:macro name="phantomx_pincher_joint" params="
-     parent
-     child
-     joint_name
-     joint_type
-     joint_origin_xyz
-     joint_origin_rpy
-     joint_axis_xyz:=unset
-     joint_lower_limit:=unset
-     joint_upper_limit:=unset
-     joint_velocity_limit:=unset
-     joint_torque_limit:=unset
-     joint_damping:=0.0
-     joint_friction:=0.0
-     mimic_joint:=none
-     mimic_multiplier:=1.0
-     mimic_offset:=0.0
-     safety_limits:=false
+  <xacro:macro name="phantomx_pincher_joint" params="
+    parent
+    child
+    joint_name
+    joint_type
+    joint_origin_xyz
+    joint_origin_rpy
+    joint_axis_xyz:=unset
+    joint_lower_limit:=unset
+    joint_upper_limit:=unset
+    joint_velocity_limit:=unset
+    joint_torque_limit:=unset
+    joint_damping:=0.0
+    joint_friction:=0.0
+    mimic_joint:=none
+    mimic_multiplier:=1.0
+    mimic_offset:=0.0
+    safety_limits:=false
     safety_position_margin:=0.0
     safety_k_position:=0.0
