Commit message: fix: convertir DAE a STL binario — RViz no puede cargar COLLADA en este sistema

File: Laboratorio No. 05 - Robótica de Desarrollo ROS Jazzy y Phantom Pincher X100/pincher_description/urdf/phantomx_pincher_utils.xacro (robot description, xacro)
@@ -32,5 +32,5 @@
         <origin xyz="${mesh_offset_visual_xyz}" rpy="${mesh_offset_visual_rpy}"/>
         <geometry>
-          <mesh filename="package://pincher_description/meshes/visual/${mesh}.dae"/>
+          <mesh filename="package://pincher_description/meshes/visual/${mesh}.stl"/>
         </geometry>
       </visual>

Commit message: fix: restaurar .dae para visual (STL convertido tenia orientacion rota) + corregir collision.stl

File: Laboratorio No. 05 - Robótica de Desarrollo ROS Jazzy y Phantom Pincher X100/pincher_description/urdf/phantomx_pincher_utils.xacro (robot description, xacro)
@@ -32,5 +32,5 @@
         <origin xyz="${mesh_offset_visual_xyz}" rpy="${mesh_offset_visual_rpy}"/>
         <geometry>
-          <mesh filename="package://pincher_description/meshes/visual/${mesh}.stl"/>
+          <mesh filename="package://pincher_description/meshes/visual/${mesh}.dae"/>
         </geometry>
       </visual>
