Commit message: fix: eliminar link world, usar base_link como raiz — coincide con el modelo original del target

File: Laboratorio No. 05 - Robótica de Desarrollo ROS Jazzy y Phantom Pincher X100/pincher_description/urdf/phantomx_pincher.urdf.xacro (robot description, xacro)
@@ -38,13 +38,7 @@
   <!--            -->
   <xacro:property name="base_link" value="base_link"/>
-  <link name="world"/>
   <!--       -->
   <!-- Robot -->
   <!--       -->
-  <joint name="world_to_pincher_joint" type="fixed">
-    <parent link="world"/>
-    <child link="$(arg prefix)${base_link}"/>
-    <origin xyz="0 0 0" rpy="0 0 0"/>
-  </joint>
   <!-- Base link that can be used for fixing the robot to the world -->
   <xacro:phantomx_pincher_dummy_link

Commit message: fix: reconectar mimic de dedos al gripper con rango [0, 0.0158] + lower limit 0

File: Laboratorio No. 05 - Robótica de Desarrollo ROS Jazzy y Phantom Pincher X100/pincher_description/urdf/phantomx_pincher.urdf.xacro (robot description, xacro)
@@ -31,5 +31,5 @@
   <xacro:arg name="ros2_controller_parameters" default=""/>
   <!-- Flag to enable mimicking of the finger joints -->
-  <xacro:arg name="mimic_finger_joints" default="false"/>
+  <xacro:arg name="mimic_finger_joints" default="true"/>
   <!-- Flag to preserve fixed joints and prevent lumping when generating SDF for Gazebo -->
   <xacro:arg name="gazebo_preserve_fixed_joint" default="false"/>

File: Laboratorio No. 05 - Robótica de Desarrollo ROS Jazzy y Phantom Pincher X100/pincher_description/urdf/phantomx_pincher_arm.xacro (robot description, xacro)
@@ -65,5 +65,5 @@
     <xacro:dynamixel_ax12_fixed prefix="${prefix}" parent="arm_wrist_F3_0_link" name="gripper_servo" joint_origin_xyz="0.0 0.0 ${-ax12_width/2}" joint_origin_rpy="${pi/2} ${pi} ${pi/2}" collision="${collision}" gazebo_preserve_fixed_joint="${gazebo_preserve_fixed_joint}"/>
     <xacro:gripper_finger_base prefix="${prefix}" parent="gripper_servo_link" name="gripper_finger_base" joint_origin_xyz="0 ${ax12_width/2} 0.0" joint_origin_rpy="${pi} 0.0 ${pi/2}" collision="${collision}" gazebo_preserve_fixed_joint="${gazebo_preserve_fixed_joint}"/>
-    <xacro:pincher_finger prefix="${prefix}" parent="gripper_finger_base_link" name="gripper_finger1" joint_origin_xyz="${finger_centre_offset_x} ${finger_centre_offset_y} 0.0" joint_origin_rpy="${pi/2} 0.0 ${pi/2}" collision="${collision}" gazebo_preserve_fixed_joint="${gazebo_preserve_fixed_joint}"/>
+    <xacro:pincher_finger prefix="${prefix}" parent="gripper_finger_base_link" name="gripper_finger1" joint_origin_xyz="${finger_centre_offset_x} ${finger_centre_offset_y} 0.0" joint_origin_rpy="${pi/2} 0.0 ${pi/2}" collision="${collision}" gazebo_preserve_fixed_joint="${gazebo_preserve_fixed_joint}" mimic_joint="${prefix}gripper" mimic_multiplier="0.00503" mimic_offset="0.0079"/>
     <!-- If enabled, mimic finger joints -->
     <xacro:if value="${mimic_finger_joints}">

File: Laboratorio No. 05 - Robótica de Desarrollo ROS Jazzy y Phantom Pincher X100/pincher_description/urdf/phantomx_pincher_hardware.xacro (robot description, xacro)
@@ -180,5 +180,5 @@
   <xacro:property name="pincher_finger_joint_type" value="prismatic"/>
   <xacro:property name="pincher_finger_joint_axis_xyz" value="1.0 0.0 0.0"/>
-  <xacro:property name="pincher_finger_joint_lower_limit" value="0.001"/>
+  <xacro:property name="pincher_finger_joint_lower_limit" value="0.0"/>
   <xacro:property name="pincher_finger_joint_upper_limit" value="0.0158"/>
   <xacro:property name="pincher_finger_joint_velocity_limit" value="0.01"/>

Commit message: fix: rotar brazo a vertical (rpy 0 -pi/2 0 en kit_to_arm_base_joint)

File: Laboratorio No. 05 - Robótica de Desarrollo ROS Jazzy y Phantom Pincher X100/pincher_description/urdf/phantomx_pincher.urdf.xacro (robot description, xacro)
@@ -59,6 +59,6 @@
     <!-- Child: base link of the PhantomX arm -->
     <child link="$(arg prefix)arm_base_link"/>
-    <!-- Pose of the arm base relative to the kit (tuned in original repo) -->
-    <origin xyz="0.01325 0 0.016" rpy="0 0 0"/>
+    <!-- Rotate arm to vertical (matches global_rotation_rpy from kit.xacro) -->
+    <origin xyz="0.01325 0 0.016" rpy="0 ${-pi/2} 0"/>
   </joint>
   <!-- Arm -->

Commit message: fix: revertir todo a original excepto shoulder rpy=0 pi/2 0 que apunta arriba

File: Laboratorio No. 05 - Robótica de Desarrollo ROS Jazzy y Phantom Pincher X100/pincher_description/urdf/phantomx_pincher.urdf.xacro (robot description, xacro)
@@ -59,6 +59,6 @@
     <!-- Child: base link of the PhantomX arm -->
     <child link="$(arg prefix)arm_base_link"/>
-    <!-- Rotate arm to vertical (matches global_rotation_rpy from kit.xacro) -->
-    <origin xyz="0.01325 0 0.016" rpy="0 ${-pi/2} 0"/>
+    <!-- Pose of the arm base relative to the kit (tuned in original repo) -->
+    <origin xyz="0.01325 0 0.016" rpy="0 0 0"/>
   </joint>
   <!-- Arm -->

File: Laboratorio No. 05 - Robótica de Desarrollo ROS Jazzy y Phantom Pincher X100/pincher_description/urdf/phantomx_pincher_arm.xacro (robot description, xacro)
@@ -42,5 +42,5 @@
     <link name="${prefix}${base_link}"/>
     <!-- Shoulder Pan -->
-    <xacro:dynamixel_ax12_fixed prefix="${prefix}" parent="${base_link}" name="arm_shoulder_pan_servo" joint_origin_xyz="0.0 0.0 0.0" joint_origin_rpy="${pi/2} ${-pi/2} ${pi/2}" collision="${collision}" gazebo_preserve_fixed_joint="${gazebo_preserve_fixed_joint}"/>
+    <xacro:dynamixel_ax12_fixed prefix="${prefix}" parent="${base_link}" name="arm_shoulder_pan_servo" joint_origin_xyz="0.0 0.0 0.0" joint_origin_rpy="${pi/2} 0.0 ${pi/2}" collision="${collision}" gazebo_preserve_fixed_joint="${gazebo_preserve_fixed_joint}"/>
     <xacro:bioloid_f3_revolute prefix="${prefix}" parent="arm_shoulder_pan_servo_link" name="waist" joint_velocity_limit="${joints_velocity_limit}" joint_lower_limit="${pan_joint_lower_limit}" joint_upper_limit="${pan_joint_upper_limit}" joint_origin_xyz="0 ${ax12_width/2} 0.0" joint_origin_rpy="${-pi/2} ${pi/2} ${pi}" collision="${collision}" gazebo_preserve_fixed_joint="${gazebo_preserve_fixed_joint}"/>
     <!-- Shoulder Lift -->
