Commit message: fix: corregir package://phantomx_pincher_description → pincher_description en kit.xacro y utils.xacro

File: Laboratorio No. 05 - Robótica de Desarrollo ROS Jazzy y Phantom Pincher X100/pincher_description/urdf/kit.xacro (robot description, xacro)
@@ -28,5 +28,5 @@
       <origin xyz="0.155 0 0.000" rpy="0 0 -${PI/2}" />
       <geometry>
-        <mesh filename="package://phantomx_pincher_description/meshes/STL/baseElementosFijos.stl"
+        <mesh filename="package://pincher_description/meshes/STL/baseElementosFijos.stl"
               scale="0.001 0.001 0.001" />
       </geometry>
@@ -45,5 +45,5 @@
       <origin xyz="0 0 0" rpy="${PI} 0 ${PI/2}" />
       <geometry>
-        <mesh filename="package://phantomx_pincher_description/meshes/STL/caseBaseRobot.stl"
+        <mesh filename="package://pincher_description/meshes/STL/caseBaseRobot.stl"
               scale="0.001 0.001 0.001" />
       </geometry>
@@ -67,5 +67,5 @@
       <origin xyz="0.155 0 0" rpy="0 0 0" />
       <geometry>
-        <mesh filename="package://phantomx_pincher_description/meshes/STL/canastilla.stl"
+        <mesh filename="package://pincher_description/meshes/STL/canastilla.stl"
               scale="0.001 0.001 0.001" />
       </geometry>
@@ -110,5 +110,5 @@
       <origin xyz="0.26028 0 0" rpy="0 0 -${PI/2}" />
       <geometry>
-        <mesh filename="package://phantomx_pincher_description/meshes/STL/ensambleSoporteCamara.stl"
+        <mesh filename="package://pincher_description/meshes/STL/ensambleSoporteCamara.stl"
               scale="0.001 0.001 0.001" />
       </geometry>
@@ -132,5 +132,5 @@
       <origin xyz="0 0 0" rpy="${PI} 0 0" />
       <geometry>
-        <mesh filename="package://phantomx_pincher_description/meshes/STL/zonaCircular146mm.stl"
+        <mesh filename="package://pincher_description/meshes/STL/zonaCircular146mm.stl"
               scale="0.001 0.001 0.001" />
       </geometry>
@@ -154,5 +154,5 @@
       <origin xyz="0 0 0" rpy="${PI/2} 0 -${PI/2}" />
       <geometry>
-        <mesh filename="package://phantomx_pincher_description/meshes/STL/ensambleAirpump.stl"
+        <mesh filename="package://pincher_description/meshes/STL/ensambleAirpump.stl"
               scale="0.001 0.001 0.001" />
       </geometry>
@@ -176,5 +176,5 @@
       <origin xyz="0 0 0" rpy="-${PI/2} 0 ${PI/2}" />
       <geometry>
-        <mesh filename="package://phantomx_pincher_description/meshes/STL/manija.stl"
+        <mesh filename="package://pincher_description/meshes/STL/manija.stl"
               scale="0.001 0.001 0.001" />
       </geometry>
@@ -198,5 +198,5 @@
       <origin xyz="0 0 0" rpy="-${PI/2} 0 ${PI/2}" />
       <geometry>
-        <mesh filename="package://phantomx_pincher_description/meshes/STL/manija.stl"
+        <mesh filename="package://pincher_description/meshes/STL/manija.stl"
               scale="0.001 0.001 0.001" />
       </geometry>
@@ -220,5 +220,5 @@
       <origin xyz="0 0 0" rpy="0 0 -${PI/2}" />
       <geometry>
-        <mesh filename="package://phantomx_pincher_description/meshes/STL/canecaGrande.stl"
+        <mesh filename="package://pincher_description/meshes/STL/canecaGrande.stl"
               scale="0.001 0.001 0.001" />
       </geometry>
@@ -228,5 +228,5 @@
       <origin xyz="0 0 0" rpy="0 0 -${PI/2}" />
       <geometry>
-        <mesh filename="package://phantomx_pincher_description/meshes/STL/canecaGrande.stl"
+        <mesh filename="package://pincher_description/meshes/STL/canecaGrande.stl"
               scale="0.001 0.001 0.001" />
       </geometry>
@@ -243,5 +243,5 @@
       <origin xyz="0 0 0" rpy="0 0 ${PI/2}" />
       <geometry>
-        <mesh filename="package://phantomx_pincher_description/meshes/STL/canecaGrande.stl"
+        <mesh filename="package://pincher_description/meshes/STL/canecaGrande.stl"
               scale="0.001 0.001 0.001" />
       </geometry>
@@ -251,5 +251,5 @@
       <origin xyz="0 0 0" rpy="0 0 ${PI/2}" />
       <geometry>
-        <mesh filename="package://phantomx_pincher_description/meshes/STL/canecaGrande.stl"
+        <mesh filename="package://pincher_description/meshes/STL/canecaGrande.stl"
               scale="0.001 0.001 0.001" />
       </geometry>
@@ -266,5 +266,5 @@
       <origin xyz="0 0 0" rpy="0 0 ${PI*((180-25.5)/180)}" />
       <geometry>
-        <mesh filename="package://phantomx_pincher_description/meshes/STL/canecaGrande.stl"
+        <mesh filename="package://pincher_description/meshes/STL/canecaGrande.stl"
               scale="0.001 0.001 0.001" />
       </geometry>
@@ -274,5 +274,5 @@
       <origin xyz="0 0 0" rpy="0 0 ${PI*((180-25.5)/180)}" />
       <geometry>
-        <mesh filename="package://phantomx_pincher_description/meshes/STL/canecaGrande.stl"
+        <mesh filename="package://pincher_description/meshes/STL/canecaGrande.stl"
               scale="0.001 0.001 0.001" />
       </geometry>
@@ -289,5 +289,5 @@
       <origin xyz="0 0 0" rpy="0 0 ${PI*(25.5/180) + PI}" />
       <geometry>
-        <mesh filename="package://phantomx_pincher_description/meshes/STL/canecaGrande.stl"
+        <mesh filename="package://pincher_description/meshes/STL/canecaGrande.stl"
               scale="0.001 0.001 0.001" />
       </geometry>
@@ -297,5 +297,5 @@
       <origin xyz="0 0 0" rpy="0 0 ${PI*(25.5/180) + PI}" />
       <geometry>
-        <mesh filename="package://phantomx_pincher_description/meshes/STL/canecaGrande.stl"
+        <mesh filename="package://pincher_description/meshes/STL/canecaGrande.stl"
               scale="0.001 0.001 0.001" />
       </geometry>

File: Laboratorio No. 05 - Robótica de Desarrollo ROS Jazzy y Phantom Pincher X100/pincher_description/urdf/phantomx_pincher_utils.xacro (robot description, xacro)
@@ -32,5 +32,5 @@
         <origin xyz="${mesh_offset_visual_xyz}" rpy="${mesh_offset_visual_rpy}"/>
         <geometry>
-          <mesh filename="package://phantomx_pincher_description/meshes/visual/${mesh}.dae"/>
+          <mesh filename="package://pincher_description/meshes/visual/${mesh}.dae"/>
         </geometry>
       </visual>
@@ -40,5 +40,5 @@
           <geometry>
             <xacro:if value="${collision_type == 'mesh'}">
-              <mesh filename="package://phantomx_pincher_description/meshes/collision/${mesh}.stl"/>
+              <mesh filename="package://pincher_description/meshes/collision/${mesh}.stl"/>
             </xacro:if>
             <xacro:if value="${collision_type == 'box'}">

Commit message: fix: aplicar global_rotation_rpy (0, -pi/2, 0) para que home sea vertical

File: Laboratorio No. 05 - Robótica de Desarrollo ROS Jazzy y Phantom Pincher X100/pincher_description/urdf/kit.xacro (robot description, xacro)
@@ -315,5 +315,5 @@
     <parent link="world_link"/>
     <child link="baseFija_link"/>
-    <origin xyz="0 0 0" rpy="0 0 0" />
+    <origin xyz="0 0 0" rpy="${global_rotation_rpy}" />
   </joint>
   <!--

Commit message: fix: rotar shoulder -90° en X para que home sea vertical (revertir global_rotation)

File: Laboratorio No. 05 - Robótica de Desarrollo ROS Jazzy y Phantom Pincher X100/pincher_description/urdf/kit.xacro (robot description, xacro)
@@ -315,5 +315,5 @@
     <parent link="world_link"/>
     <child link="baseFija_link"/>
-    <origin xyz="0 0 0" rpy="${global_rotation_rpy}" />
+    <origin xyz="0 0 0" rpy="0 0 0" />
   </joint>
   <!--

File: Laboratorio No. 05 - Robótica de Desarrollo ROS Jazzy y Phantom Pincher X100/pincher_description/urdf/phantomx_pincher_arm.xacro (robot description, xacro)
@@ -46,5 +46,5 @@
     <!-- Shoulder Lift -->
     <xacro:dynamixel_ax12_fixed prefix="${prefix}" parent="waist_link" name="arm_shoulder_lift_servo" joint_origin_xyz="0.0 0.0 ${-ax12_height-f10_height+0.001}" joint_origin_rpy="0.0 ${pi} 0.0" collision="${collision}" gazebo_preserve_fixed_joint="${gazebo_preserve_fixed_joint}"/>
-    <xacro:bioloid_f4_revolute prefix="${prefix}" parent="arm_shoulder_lift_servo_link" name="shoulder" joint_velocity_limit="${joints_velocity_limit}" joint_lower_limit="${shoulder_joint_lower_limit}" joint_upper_limit="${shoulder_joint_upper_limit}" joint_origin_xyz="0.0 0.0 0.0" joint_origin_rpy="0.0 0.0 0.0" collision="${collision}" gazebo_preserve_fixed_joint="${gazebo_preserve_fixed_joint}"/>
+    <xacro:bioloid_f4_revolute prefix="${prefix}" parent="arm_shoulder_lift_servo_link" name="shoulder" joint_velocity_limit="${joints_velocity_limit}" joint_lower_limit="${shoulder_joint_lower_limit}" joint_upper_limit="${shoulder_joint_upper_limit}" joint_origin_xyz="0.0 0.0 0.0" joint_origin_rpy="${-pi/2} 0.0 0.0" collision="${collision}" gazebo_preserve_fixed_joint="${gazebo_preserve_fixed_joint}"/>
     <xacro:bioloid_f10_fixed prefix="${prefix}" parent="shoulder_link" name="arm_shoulder_F10_0" joint_origin_xyz="0.0 0.0 ${f4_height+f10_height/2}" joint_origin_rpy="0.0 0.0 0.0" collision="${collision}" gazebo_preserve_fixed_joint="${gazebo_preserve_fixed_joint}"/>
     <xacro:bioloid_f10_fixed prefix="${prefix}" parent="arm_shoulder_F10_0_link" name="arm_shoulder_F10_1" joint_origin_xyz="0.0 0.0 ${f10_height}" joint_origin_rpy="0.0 0.0 0.0" collision="${collision}" gazebo_preserve_fixed_joint="${gazebo_preserve_fixed_joint}"/>

Commit message: fix: quitar canastilla del modelo

File: Laboratorio No. 05 - Robótica de Desarrollo ROS Jazzy y Phantom Pincher X100/pincher_description/urdf/kit.xacro (robot description, xacro)
@@ -62,47 +62,4 @@
     <child link="caseBaseRobot_link" />
     <origin xyz="-0.01325 0 0.054" rpy="0 0 0" />
-  </joint>
-  <link name="canastilla_link">
-    <visual>
-      <origin xyz="0.155 0 0" rpy="0 0 0" />
-      <geometry>
-        <mesh filename="package://pincher_description/meshes/STL/canastilla.stl"
-              scale="0.001 0.001 0.001" />
-      </geometry>
-      <material name="blue" />
-    </visual>
-    <collision>
-        <origin xyz="-0.1365 0.0 0.0905" rpy="0 0 0" />
-        <geometry>
-            <box size="0.017 0.4 0.1855" />
-        </geometry>
-        <material name="blue" />
-    </collision>
-    <collision>
-        <origin xyz="0.4465 0.0 0.0905" rpy="0 0 0" />
-        <geometry>
-            <box size="0.017 0.4 0.1855" />
-        </geometry>
-        <material name="blue" />
-    </collision>
-    <collision>
-        <origin xyz="0.155 0.1915 0.0905" rpy="0 0 0" />
-        <geometry>
-            <box size="0.6 0.017 0.1855" />
-        </geometry>
-        <material name="blue" />
-    </collision>
-    <collision>
-        <origin xyz="0.155 -0.1915 0.0905" rpy="0 0 0" />
-        <geometry>
-            <box size="0.6 0.017 0.1855" />
-        </geometry>
-        <material name="blue" />
-    </collision>
-  </link>
-  <joint name="base_canastilla_joint" type="fixed">
-    <parent link="baseFija_link" />
-    <child link="canastilla_link" />
-    <origin xyz="0 0 0" rpy="0 0 0" />
   </joint>
   <link name="ensambleSoporteCamara_link">
